File: Ebox/Ebox.kicad_sch (KiCad schematic)
At the start: 3 parts, among them J1 Screw_Terminal_01x12, J2 Screw_Terminal_01x12

Commit message: updated Arm arduino code, manual_operate, and PCBs
Parts:
- added J3: Screw_Terminal_01x04, TerminalBlock_Phoenix:TerminalBlock_Phoenix_MPT-0,5-4-2.54_1x04_P2.54mm_Horizontal, symbol Connector:Screw_Terminal_01x04
- added J4: Screw_Terminal_01x02, TerminalBlock_TE-Connectivity:TerminalBlock_TE_282834-2_1x02_P2.54mm_Horizontal, symbol Connector:Screw_Terminal_01x02
- added M1, M2, M3: MNMOS, IRF520:TO270P460X1020X2008-3P, symbol pspice:MNMOS
Connections:
- net at XA1.D26: now also M3.2 (G)
- net at XA1.D27: now also M2.2 (G)
- net at XA1.D28: now also M1.2 (G)
- new net: J4.1 (Pin_1), M1.1 (D), M2.1 (D), M3.1 (D)
- new net: J3.4 (Pin_4), M1.3 (S)
- new net: J3.1 (Pin_1), J4.2 (Pin_2)
- new net: J3.2 (Pin_2), M3.3 (S), M3.4 (B)
- new net: J3.3 (Pin_3), M2.3 (S)
