File: Science/Science.kicad_sch (KiCad schematic)
At the start: 4 parts, among them J1 Screw_Terminal_01x12, J2 Screw_Terminal_01x12, U1 LM1084-5.0

Commit message: Updated Arduino README.. still needs more
Parts:
- added D1, D2: LED, LED_SMD:LED-APA102-2020, symbol Device:LED
- added R1, R2: R_US, Resistor_SMD:R_0201_0603Metric, symbol Device:R_US
Connections:
- net GND: now also D1.1 (K), D2.1 (K)
- net at A1.1 (D1/TX): now also R2.1
- net at A1.2 (D0/RX): now also R1.1
- new net: D2.2 (A), R2.2
- new net: D1.2 (A), R1.2
