File: Arm/lowerArm_upperArm/lowerArm.kicad_sch (KiCad schematic)
At the start: 14 parts, among them J1 Screw_Terminal_01x12, J2 Screw_Terminal_01x12, J3 Screw_Terminal_01x02, U1 LM1084-5.0, U2 Crystal_Oscillator_8MHz, U3 MCP2515-xSO, U4 MAX3051

Commit message: Added Teensy programs to Microcontrollers folder
Other:
- note added: "2023 Capstone Arm Motor Controller PCBS"
- note added: "3/9/2023"
- note added: "By: Jack Cornette"
- note added: "Lower and Upper Arm PCB"
- note removed: "- arduino Nano - screw terminals - 5v regulator - CAN stuff (connect to screw terminals) - LED indicators (CAN set up complete, msg recieved, nano has 1 built in LED we can use)"
Changed lines of the file:
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@@
     (stroke (width 0) (type default) (color 0 0 0 0))
   )
-  (text "- arduino Nano\n- screw terminals\n- 5v regulator\n- CAN stuff (connect to screw terminals)\n- LED indicators (CAN set up complete, msg recieved, nano has 1 built in LED we can use)"
-    (at 15.24 25.4 0)
+  (text "3/9/2023" (at 207.01 194.31 0)
     (effects (font (size 1.27 1.27)) (justify left bottom))
   )
+  (text "Lower and Upper Arm PCB" (at 179.07 179.07 0)
+    (effects (font (size 5 5)) (justify left bottom))
+  )
+  (text "2023 Capstone Arm Motor Controller PCBS" (at 186.69 190.5 0)
+    (effects (font (size 1.27 1.27)) (justify left bottom))
+  )
+  (text "By: Jack Cornette" (at 264.16 190.5 0)
+    (effects (font (size 1.27 1.27)) (justify left bottom))
+  )
